File: Electronics/uSD2PSX/rp2040-memcard.kicad_pcb (KiCad board)
At the start: 2 copper layers, 24 x 32 mm, 40 parts, among them J101 PS2, J102 BSEL, J103 GND, J104 3V3, J105 SCL, J106 SDA, J107 SWC, J108 SWD, J110 DP, J111 DN, J112 GND, J113 3V3, J114 MEM2085-00-115-00-A_REV0.2, U101 W25Q16JVUXIQ, U102 RP2040, U4 LY68L6400SLIT, Y101 12MHz

Commit message: correct part number of uSD2PSX SPI flash
Parts:
- U101: value W25Q16JVUXIQ -> W25Q128JVPIQ
Changed lines of the file:
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@@
     (descr "WSON, 8 Pin (http://www.winbond.com/resource-files/w25q32jv%20revg%2003272018%20plus.pdf (page 68)), generated with kicad-footprint-generator ipc_noLead_generator.py")
     (tags "WSON NoLead")
-    (property "Part Number" "W25Q16JVUXIQ TR")
+    (property "Part Number" "W25Q128JVPIQ")
     (property "Sheetfile" "rp2040-memcard.kicad_sch")
     (property "Sheetname" "")
@@
         (effects (font (size 1 1) (thickness 0.15)))
     )
-    (fp_text value "W25Q16JVUXIQ" (at 0 3.45 90) (layer "F.Fab")
+    (fp_text value "W25Q128JVPIQ" (at 0 3.45 90) (layer "F.Fab")
         (effects (font (size 1 1) (thickness 0.15)))
     )
