File: Electronics/PS2_79004_Rev_0_4/MechaCon_Interfaces.kicad_sch (KiCad schematic)
At the start: 76 parts, among them SW101 SW_Push, U106 APX811-31UG, U1401 CXR726080, Y1501 32.768kHz, Y1502 16,934MHz

Commit message: Update part number of crystal Y1502 on REF4000
Parts:
- Y1502: Part Number NX3225GA-16.9344M-STD-CRG-2‎ -> STDCRG2-16.9344M
Changed lines of the file:
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@@
       (effects (font (size 1.27 1.27)) hide)
     )
-    (property "Part Number" "NX3225GA-16.9344M-STD-CRG-2‎" (at 172.72 231.14 0)
+    (property "Part Number" "STDCRG2-16.9344M" (at 172.72 231.14 0)
       (effects (font (size 1.27 1.27)) hide)
     )
