File: Electronics/PS2_79004_Rev_0_4/PS2_79004_Rev_0_4.kicad_pcb (KiCad board)
At the start: 6 copper layers, 121 x 83 mm, 770 parts, among them J2101 LEFT SPEAKER, J2102 RIGHT SPEAKER, J2103 SJ-43504-SMT-TR, J2501 Conn_01x40_MountingPin, J3001 EXPANSION HDR, J3002 ETH, J3003 USB_A, J3004 GAMEPAD LEFT, J3005 GAMEPAD RIGHT, J3006 Debug, J3007 2328702-4, J301 BAT1, J302 BAT2, P201 CX90MW6-16P, Q201 Q_SI7223DN, Q301 CSD17575Q3, Q302 CSD17575Q3, Q303 CSD17575Q3, Q401 DMN67D8L, Q402 DMN67D8L, Q403 BSS84AK, Q601 DMN67D8L, U1401 CXR726080, U1501 APX811-31UG, U1601 LM20BIM7, U1701 74LVC1G08, U1702 74LVC1G08, U1703 S29JL064J55TFI000, U1801 CXD3098AQ, U2001 BCM5241, U201 TVS2200DRV, U202 STUSB4500, U203 TXS0102DQE, U2101 TXS0102DQE, U2102 74LVC1G07, U2103 LM49450, U2201 CXD2980, U2501 TPS92360, U2601 T20F256I4, U2701 APX811-31UG, U2801 IS45S32400F, U301 BQ25792B, U302 MAX17320, U501 MPQ8626GD, U502 TPS629210, U503 TPS629210, U504 TPS629210, U505 TPS629210, U506 AP22653A, U507 TLV75525PDRV, U508 TLV75518PDRV, U509 TLV75518PDRV, U601 74LVC1G07, U602 W25Q128JVPIQ, U603 RP2040, U801 627G04LF, U901 CXD2976GB, X2901 ASE-50MHz, Y1501 32.768kHz, Y1502 16,934MHz, Y601 12MHz, Y801 18.432MHz

Commit message: Update part number of crystal Y1502 on REF4000
Connections:
- net /Connectors/CRESET_N renamed /System Controller/T20_CRESET
Changed lines of the file:
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@@
   (net 565 "unconnected-(U901J-NC-PadD3)")
   (net 566 "/System Controller/USB_IN_DN")
-  (net 567 "/Connectors/CRESET_N")
+  (net 567 "/System Controller/T20_CRESET")
   (net 568 "/PlayStation 2 - MAIN/Audio/LS+")
   (net 569 "/PlayStation 2 - MAIN/Audio/LS-")
@@
       (net 232 "Net-(U2701-~{RESET})") (pintype "passive"))
     (pad "2" smd roundrect (at 0.51 0) (size 0.54 0.64) (layers "F.Cu" "F.Paste" "F.Mask") (roundrect_rratio 0.25)
-      (net 567 "/Connectors/CRESET_N") (pintype "passive"))
+      (net 567 "/System Controller/T20_CRESET") (pintype "passive"))
     (model "${KICAD6_3DMODEL_DIR}/Resistor_SMD.3dshapes/R_0402_1005Metric.wrl"
       (offset (xyz 0 0 0))
@@
     (descr "SMD Crystal SERIES SMD3225/4 http://www.txccrystal.com/images/pdf/7m-accuracy.pdf, 3.2x2.5mm^2 package")
     (tags "SMD SMT crystal")
-    (property "Part Number" "NX3225GA-16.9344M-STD-CRG-2‎")
+    (property "Part Number" "STDCRG2-16.9344M")
     (property "Sheetfile" "MechaCon_Interfaces.kicad_sch")
     (property "Sheetname" "Mechacon")
@@
       (net 116 "/Connectors/TMS") (pinfunction "Pin_2") (pintype "passive"))
     (pad "3" smd rect (at -1.95 -2.54 180) (size 2.4 0.74) (layers "F.Cu" "F.Paste" "F.Mask")
-      (net 567 "/Connectors/CRESET_N") (pinfunction "Pin_3") (pintype "passive"))
+      (net 567 "/System Controller/T20_CRESET") (pinfunction "Pin_3") (pintype "passive"))
     (pad "4" smd rect (at 1.95 -2.54 180) (size 2.4 0.74) (layers "F.Cu" "F.Paste" "F.Mask")
       (net 117 "/Connectors/TCK") (pinfunction "Pin_4") (pintype "passive"))
@@
       (net 531 "unconnected-(U2601D-GPIOR_154-PadN16)") (pinfunction "GPIOR_154") (pintype "bidirectional+no_connect"))
     (pad "P1" smd circle locked (at -6 4.4 180) (size 0.32 0.32) (layers "F.Cu" "F.Mask")
-      (net 567 "/Connectors/CRESET_N") (pinfunction "CRESET_N") (pintype "input"))
+      (net 567 "/System Controller/T20_CRESET") (pinfunction "CRESET_N") (pintype "input"))
     (pad "P2" smd circle locked (at -5.2 4.4 180) (size 0.32 0.32) (layers "F.Cu" "F.Mask")
       (net 532 "unconnected-(U2601B-GPIOL_02-PadP2)") (pinfunction "GPIOL_02") (pintype "bidirectional+no_connect"))
@@
       (net 362 "Net-(TP601-Pin_1)") (pinfunction "RUN") (pintype "input"))
     (pad "27" smd roundrect locked (at 2.2 3.4375 270) (size 0.2 0.875) (layers "F.Cu" "F.Paste" "F.Mask") (roundrect_rratio 0.25)
-      (net 567 "/Connectors/CRESET_N") (pinfunction "GPIO16") (pintype "bidirectional"))
+      (net 567 "/System Controller/T20_CRESET") (pinfunction "GPIO16") (pintype "bidirectional"))
     (pad "28" smd roundrect locked (at 2.6 3.4375 270) (size 0.2 0.875) (layers "F.Cu" "F.Paste" "F.Mask") (roundrect_rratio 0.25)
       (net 622 "/PlayStation 2 - MAIN/PS2_LED_RED") (pinfunction "GPIO17") (pintype "bidirectional"))
@@
     )
   )
-  (zone (net 567) (net_name "/Connectors/CRESET_N") (layer "F.Cu") (name "$teardrop_padvia$") (hatch edge 0.5)
+  (zone (net 567) (net_name "/System Controller/T20_CRESET") (layer "F.Cu") (name "$teardrop_padvia$") (hatch edge 0.5)
     (priority 30653)
     (attr (teardrop (type padvia)))
@@
     )
   )
-  (zone (net 567) (net_name "/Connectors/CRESET_N") (layer "F.Cu") (name "$teardrop_padvia$") (hatch edge 0.5)
+  (zone (net 567) (net_name "/System Controller/T20_CRESET") (layer "F.Cu") (name "$teardrop_padvia$") (hatch edge 0.5)
     (priority 30498)
     (attr (teardrop (type padvia)))
@@
     )
   )
-  (zone (net 567) (net_name "/Connectors/CRESET_N") (layer "F.Cu") (name "$teardrop_padvia$") (hatch edge 0.5)
+  (zone (net 567) (net_name "/System Controller/T20_CRESET") (layer "F.Cu") (name "$teardrop_padvia$") (hatch edge 0.5)
     (priority 30352)
     (attr (teardrop (type padvia)))
@@
     )
   )
-  (zone (net 567) (net_name "/Connectors/CRESET_N") (layer "In3.Cu") (name "$teardrop_padvia$") (hatch edge 0.5)
+  (zone (net 567) (net_name "/System Controller/T20_CRESET") (layer "In3.Cu") (name "$teardrop_padvia$") (hatch edge 0.5)
     (priority 30044)
     (attr (teardrop (type padvia)))
@@
     )
   )
-  (zone (net 567) (net_name "/Connectors/CRESET_N") (layer "In3.Cu") (name "$teardrop_padvia$") (hatch edge 0.5)
+  (zone (net 567) (net_name "/System Controller/T20_CRESET") (layer "In3.Cu") (name "$teardrop_padvia$") (hatch edge 0.5)
     (priority 30036)
     (attr (teardrop (type padvia)))
